Commit message: Making the robot move

File: src/darnet_controller_test/urdf/darnetnew.xacro (robot description, xacro)
@@ -1,2644 +1,2284 @@
 <?xml version="1.0" ?>
-<robot name="darnetnew" xmlns:xacro="http://www.ros.org/wiki/xacro">
-<xacro:include filename="$(find darnetnew_description)/urdf/materials.xacro" />
-<xacro:include filename="$(find darnetnew_description)/urdf/darnetnew.trans" />
-<xacro:include filename="$(find darnetnew_description)/urdf/darnetnew.gazebo" />
-<link name="base_link">
-  <inertial>
-    <origin xyz="0.11490191942179352 -0.08811411521808868 0.4285754030138091" rpy="0 0 0"/>
-    <mass value="0.04783342981131993"/>
-    <inertia ixx="0.00012" iyy="0.000191" izz="0.00024" ixy="0.0" iyz="0.0" ixz="-0.0"/>
-  </inertial>
-  <visual>
-    <origin xyz="0 0 0" rpy="0 0 0"/>
-    <geometry>
-      <mesh filename="file://$(find darnetnew_description)/meshes/base_link.stl" scale="0.001 0.001 0.001"/>
-    </geometry>
-    <material name="silver"/>
-  </visual>
-  <collision>
-    <origin xyz="0 0 0" rpy="0 0 0"/>
-    <geometry>
-      <mesh filename="file://$(find darnetnew_description)/meshes/base_link.stl" scale="0.001 0.001 0.001"/>
-    </geometry>
-  </collision>
-</link>
-<link name="BadanAtasRevisi_1">
-  <inertial>
-    <origin xyz="-0.06259339074336327 -0.06108835494549206 0.005762936141855413" rpy="0 0 0"/>
-    <mass value="0.031847275190689105"/>
-    <inertia ixx="5e-05" iyy="8.1e-05" izz="0.000121" ixy="-0.0" iyz="5e-06" ixz="-0.0"/>
-  </inertial>
-  <visual>
-    <origin xyz="-0.177798 0.034597 -0.481242" rpy="0 0 0"/>
-    <geometry>
-      <mesh filename="file://$(find darnetnew_description)/meshes/BadanAtasRevisi_1.stl" scale="0.001 0.001 0.001"/>
-    </geometry>
-    <material name="silver"/>
-  </visual>
-  <collision>
-    <origin xyz="-0.177798 0.034597 -0.481242" rpy="0 0 0"/>
-    <geometry>
-      <mesh filename="file://$(find darnetnew_description)/meshes/BadanAtasRevisi_1.stl" scale="0.001 0.001 0.001"/>
-    </geometry>
-  </collision>
-</link>
-<link name="BadanDepanRevisi_3DPrint_1">
-  <inertial>
-    <origin xyz="-0.032730061007183925 0.005663615482670779 -0.041214029177083" rpy="0 0 0"/>
-    <mass value="0.03802229773988109"/>
-    <inertia ixx="3.4e-05" iyy="9.8e-05" izz="6.4e-05" ixy="0.0" iyz="1e-06" ixz="-0.0"/>
-  </inertial>
-  <visual>
-    <origin xyz="-0.147798 0.029595 -0.483242" rpy="0 0 0"/>
-    <geometry>
-      <mesh filename="file://$(find darnetnew_description)/meshes/BadanDepanRevisi_3DPrint_1.stl" scale="0.001 0.001 0.001"/>
-    </geometry>
-    <material name="silver"/>
-  </visual>
-  <collision>
-    <origin xyz="-0.147798 0.029595 -0.483242" rpy="0 0 0"/>
-    <geometry>
-      <mesh filename="file://$(find darnetnew_description)/meshes/BadanDepanRevisi_3DPrint_1.stl" scale="0.001 0.001 0.001"/>
-    </geometry>
-  </collision>
-</link>
-<link name="TempatBatteryRevisi2_1">
-  <inertial>
-    <origin xyz="0.00017667571617335787 -0.047857480766390126 -0.038024075665795076" rpy="0 0 0"/>
-    <mass value="0.016941557534864572"/>
-    <inertia ixx="3.3e-05" iyy="9e-06" izz="3.8e-05" ixy="-0.0" iyz="-4e-06" ixz="-0.0"/>
-  </inertial>
-  <visual>
-    <origin xyz="-0.115298 0.029597 -0.404695" rpy="0 0 0"/>
-    <geometry>
-      <mesh filename="file://$(find darnetnew_description)/meshes/TempatBatteryRevisi2_1.stl" scale="0.001 0.001 0.001"/>
-    </geometry>
-    <material name="silver"/>
-  </visual>
-  <collision>
-    <origin xyz="-0.115298 0.029597 -0.404695" rpy="0 0 0"/>
-    <geometry>
-      <mesh filename="file://$(find darnetnew_description)/meshes/TempatBatteryRevisi2_1.stl" scale="0.001 0.001 0.001"/>
-    </geometry>
-  </collision>
-</link>
-<link name="SpaceMX64_2">
-  <inertial>
-    <origin xyz="0.01729959636593876 0.008613945109970225 -0.0024995396027711614" rpy="0 0 0"/>
-    <mass value="0.0036000900764554065"/>
-    <inertia ixx="1e-06" iyy="1e-06" izz="2e-06" ixy="-0.0" iyz="-0.0" ixz="0.0"/>
-  </inertial>
-  <visual>
-    <origin xyz="-0.050798 0.089597 -0.404695" rpy="0 0 0"/>
-    <geometry>
-      <mesh filename="file://$(find darnetnew_description)/meshes/SpaceMX64_2.stl" scale="0.001 0.001 0.001"/>
-    </geometry>
-    <material name="silver"/>
-  </visual>
-  <!-- <collision>
-    <origin xyz="-0.050798 0.089597 -0.404695" rpy="0 0 0"/>
-    <geometry>
-      <mesh filename="file://$(find darnetnew_description)/meshes/SpaceMX64_2.stl" scale="0.001 0.001 0.001"/>
-    </geometry>
-  </collision> -->
-</link>
-<link name="SpaceMX64_1">
-  <inertial>
-    <origin xyz="-0.017300403634061073 0.008613945109969823 -0.0024995396027708283" rpy="0 0 0"/>
-    <mass value="0.0036000900764554065"/>
-    <inertia ixx="1e-06" iyy="1e-06" izz="2e-06" ixy="-0.0" iyz="-0.0" ixz="0.0"/>
-  </inertial>
-  <visual>
-    <origin xyz="-0.179798 0.089597 -0.404695" rpy="0 0 0"/>
-    <geometry>
-      <mesh filename="file://$(find darnetnew_description)/meshes/SpaceMX64_1.stl" scale="0.001 0.001 0.001"/>
-    </geometry>
-    <material name="silver"/>
-  </visual>
-  <!-- <collision>
-    <origin xyz="-0.179798 0.089597 -0.404695" rpy="0 0 0"/>
-    <geometry>
-      <mesh filename="file://$(find darnetnew_description)/meshes/SpaceMX64_1.stl" scale="0.001 0.001 0.001"/>
-    </geometry>
-  </collision> -->
-</link>
-<link name="MX-64T_2">
-  <inertial>
-    <origin xyz="-0.01730040375965193 0.02479645502078165 -0.01745179050411727" rpy="0 0 0"/>
-    <mass value="0.07240225558380499"/>
-    <inertia ixx="3e-05" iyy="1.7e-05" izz="2.5e-05" ixy="-0.0" iyz="1e-06" ixz="0.0"/>
-  </inertial>
-  <visual>
-    <origin xyz="-0.085398 0.111597 -0.399695" rpy="0 0 0"/>
-    <geometry>
-      <mesh filename="file://$(find darnetnew_description)/meshes/MX-64T_2.stl" scale="0.001 0.001 0.001"/>
-    </geometry>
-    <material name="silver"/>
-  </visual>
-  <!-- <collision>
-    <origin xyz="-0.085398 0.111597 -0.399695" rpy="0 0 0"/>
-    <geometry>
-      <mesh filename="file://$(find darnetnew_description)/meshes/MX-64T_2.stl" scale="0.001 0.001 0.001"/>
-    </geometry>
-  </collision> -->
-</link>
-<link name="MX-64T_1">
-  <inertial>
-    <origin xyz="-0.017300403759651112 0.0027964550207814076 -0.01745179050411727" rpy="0 0 0"/>
-    <mass value="0.07240225558380499"/>
-    <inertia ixx="3e-05" iyy="1.7e-05" izz="2.5e-05" ixy="-0.0" iyz="1e-06" ixz="0.0"/>
-  </inertial>
-  <visual>
-    <origin xyz="-0.179798 0.089597 -0.399695" rpy="0 0 0"/>
-    <geometry>
-      <mesh filename="file://$(find darnetnew_description)/meshes/MX-64T_1.stl" scale="0.001 0.001 0.001"/>
-    </geometry>
-    <material name="silver"/>
-  </visual>
-  <!-- <collision>
-    <origin xyz="-0.179798 0.089597 -0.399695" rpy="0 0 0"/>
-    <geometry>
-      <mesh filename="file://$(find darnetnew_description)/meshes/MX-64T_1.stl" scale="0.001 0.001 0.001"/>
-    </geometry>
-  </collision> -->
-</link>
-<link name="PahaAtas3D_3">
-  <inertial>
-    <origin xyz="-4.036340476298861e-07 -0.0037563467783642973 -0.010402605928093445" rpy="0 0 0"/>
-    <mass value="0.008519664111309755"/>
-    <inertia ixx="6e-06" iyy="2e-06" izz="6e-06" ixy="-0.0" iyz="0.0" ixz="0.0"/>
-  </inertial>
-  <visual>
-    <origin xyz="-0.162498 0.071597 -0.359195" rpy="0 0 0"/>
-    <geometry>
-      <mesh filename="file://$(find darnetnew_description)/meshes/PahaAtas3D_3.stl" scale="0.001 0.001 0.001"/>
-    </geometry>
-    <material name="silver"/>
-  </visual>
-  <collision>
-    <mu1>1.0</mu1>
-    <mu2>1.0</mu2>
-    <kp>1e5</kp>
-    <kd>1e3</kd>
-    <origin xyz="-0.162498 0.071597 -0.359195" rpy="0 0 0"/>
-    <geometry>
-      <mesh filename="file://$(find darnetnew_description)/meshes/PahaAtas3D_3.stl" scale="0.001 0.001 0.001"/>
-    </geometry>
-  </collision>
-</link>
-<link name="PahaAtas3D_4">
-  <inertial>
-    <origin xyz="-4.0363404811560866e-07 -0.003756346778364089 -0.010402605928093445" rpy="0 0 0"/>
-    <mass value="0.008519664111309755"/>
-    <inertia ixx="6e-06" iyy="2e-06" izz="6e-06" ixy="-0.0" iyz="0.0" ixz="0.0"/>
-  </inertial>
-  <visual>
-    <origin xyz="-0.068098 0.071597 -0.359195" rpy="0 0 0"/>
-    <geometry>
-      <mesh filename="file://$(find darnetnew_description)/meshes/PahaAtas3D_4.stl" scale="0.001 0.001 0.001"/>
-    </geometry>
-    <material name="silver"/>
-  </visual>
-  <collision>
-    <origin xyz="-0.068098 0.071597 -0.359195" rpy="0 0 0"/>
-    <geometry>
-      <mesh filename="file://$(find darnetnew_description)/meshes/PahaAtas3D_4.stl" scale="0.001 0.001 0.001"/>
-    </geometry>
-  </collision>
-</link>
-<link name="6_PR13_B_SPACER_PELV_1">
-  <inertial>
-    <origin xyz="-0.015000403634035542 -0.009365366775092657 0.002499939486701186" rpy="0 0 0"/>
-    <mass value="0.0018939893916768394"/>
-    <inertia ixx="0.0" iyy="0.0" izz="1e-06" ixy="0.0" iyz="0.0" ixz="0.0"/>
-  </inertial>
-  <visual>
-    <origin xyz="-0.130298 0.067597 -0.483242" rpy="0 0 0"/>
-    <geometry>
-      <mesh filename="file://$(find darnetnew_description)/meshes/6_PR13_B_SPACER_PELV_1.stl" scale="0.001 0.001 0.001"/>
-    </geometry>
-    <material name="silver"/>
-  </visual>
-  <!-- <collision>
-    <origin xyz="-0.130298 0.067597 -0.483242" rpy="0 0 0"/>
-    <geometry>
-      <mesh filename="file://$(find darnetnew_description)/meshes/6_PR13_B_SPACER_PELV_1.stl" scale="0.001 0.001 0.001"/>
-    </geometry>
-  </collision> -->
-</link>
-<link name="MX-28AT_AR_2">
-  <inertial>
-    <origin xyz="-0.014977946179001389 -0.015783560451416226 0.015280368795609844" rpy="0 0 0"/>
-    <mass value="0.0439903769719111"/>
-    <inertia ixx="1.3e-05" iyy="8e-06" izz="1e-05" ixy="0.0" iyz="-0.0" ixz="-0.0"/>
-  </inertial>
-  <visual>
-    <origin xyz="-0.130298 0.067597 -0.488242" rpy="0 0 0"/>
-    <geometry>
-      <mesh filename="file://$(find darnetnew_description)/meshes/MX-28AT_AR_2.stl" scale="0.001 0.001 0.001"/>
-    </geometry>
-    <material name="silver"/>
-  </visual>
-  <!-- <collision>
-    <origin xyz="-0.130298 0.067597 -0.488242" rpy="0 0 0"/>
-    <geometry>
-      <mesh filename="file://$(find darnetnew_description)/meshes/MX-28AT_AR_2.stl" scale="0.001 0.001 0.001"/>
-    </geometry>
-  </collision> -->
-</link>
-<link name="2_FR07_H104_1">
-  <inertial>
-    <origin xyz="2.0685672843662184e-06 -0.0010218695419875051 0.006993834055332382" rpy="0 0 0"/>
-    <mass value="0.004611932609017796"/>
-    <inertia ixx="1e-06" iyy="2e-06" izz="2e-06" ixy="-0.0" iyz="-0.0" ixz="-0.0"/>
-  </inertial>
-  <visual>
-    <origin xyz="-0.115298 0.072097 -0.525167" rpy="0 0 0"/>
-    <geometry>
-      <mesh filename="file://$(find darnetnew_description)/meshes/2_FR07_H104_1.stl" scale="0.001 0.001 0.001"/>
-    </geometry>
-    <material name="silver"/>
-  </visual>
-  <!-- <collision>
-    <origin xyz="-0.115298 0.072097 -0.525167" rpy="0 0 0"/>
-    <geometry>
-      <mesh filename="file://$(find darnetnew_description)/meshes/2_FR07_H104_1.stl" scale="0.001 0.001 0.001"/>
-    </geometry>
-  </collision> -->
-</link>
-<link name="MX-28AT_AR_4">
-  <inertial>
-    <origin xyz="-0.0202199743251381 -2.2524917938762656e-05 0.01128343247522512" rpy="0 0 0"/>
-    <mass value="0.0439903769719111"/>
-    <inertia ixx="1e-05" iyy="1.3e-05" izz="8e-06" ixy="0.0" iyz="0.0" ixz="0.0"/>
-  </inertial>
-  <visual>
-    <origin xyz="-0.135798 0.072097 -0.553167" rpy="0 0 0"/>
-    <geometry>
-      <mesh filename="file://$(find darnetnew_description)/meshes/MX-28AT_AR_4.stl" scale="0.001 0.001 0.001"/>
-    </geometry>
-    <material name="silver"/>
-  </visual>
-  <!-- <collision>
-    <origin xyz="-0.135798 0.072097 -0.553167" rpy="0 0 0"/>
-    <geometry>
-      <mesh filename="file://$(find darnetnew_description)/meshes/MX-28AT_AR_4.stl" scale="0.001 0.001 0.001"/>
-    </geometry>
-  </collision> -->
-</link>
-<link name="MX-28AT_AR_3">
-  <inertial>
-    <origin xyz="0.014719927512307426 -0.015783560451416087 0.015022636486481222" rpy="0 0 0"/>
-    <mass value="0.0439903769719111"/>
-    <inertia ixx="1e-05" iyy="8e-06" izz="1.3e-05" ixy="0.0" iyz="0.0" ixz="0.0"/>
-  </inertial>
-  <visual>
-    <origin xyz="-0.046524 0.067597 -0.487315" rpy="0 0 0"/>
-    <geometry>
-      <mesh filename="file://$(find darnetnew_description)/meshes/MX-28AT_AR_3.stl" scale="0.001 0.001 0.001"/>
-    </geometry>
-    <material name="silver"/>
-  </visual>
-  <!-- <collision>
-    <origin xyz="-0.046524 0.067597 -0.487315" rpy="0 0 0"/>
-    <geometry>
-      <mesh filename="file://$(find darnetnew_description)/meshes/MX-28AT_AR_3.stl" scale="0.001 0.001 0.001"/>
-    </geometry>
-  </collision> -->
-</link>
-<link name="10_FR07_H102_3">
-  <inertial>
-    <origin xyz="-0.006061207664907364 -6.755027122384849e-08 -0.0026281000205751748" rpy="0 0 0"/>
-    <mass value="0.004952092458780469"/>
-    <inertia ixx="2e-06" iyy="1e-06" izz="2e-06" ixy="-0.0" iyz="0.0" ixz="-0.0"/>
-  </inertial>
-  <visual>
-    <origin xyz="-0.038174 0.072097 -0.502315" rpy="0 0 0"/>
-    <geometry>
-      <mesh filename="file://$(find darnetnew_description)/meshes/10_FR07_H102_3.stl" scale="0.001 0.001 0.001"/>
-    </geometry>
-    <material name="silver"/>
-  </visual>
-  <!-- <collision>
-    <origin xyz="-0.038174 0.072097 -0.502315" rpy="0 0 0"/>
-    <geometry>
-      <mesh filename="file://$(find darnetnew_description)/meshes/10_FR07_H102_3.stl" scale="0.001 0.001 0.001"/>
-    </geometry>
-  </collision> -->
-</link>
-<link name="MX-28AT_AR_6">
-  <inertial>
-    <origin xyz="-2.2100633829229277e-05 -0.020219638153982887 -0.011283313957089425" rpy="0 0 0"/>
-    <mass value="0.0439903769719111"/>
-    <inertia ixx="1.3e-05" iyy="1e-05" izz="8e-06" ixy="0.0" iyz="-0.0" ixz="-0.0"/>
-  </inertial>
-  <visual>
-    <origin xyz="-0.015674 0.051597 -0.486315" rpy="0 0 0"/>
-    <geometry>
-      <mesh filename="file://$(find darnetnew_description)/meshes/MX-28AT_AR_6.stl" scale="0.001 0.001 0.001"/>
-    </geometry>
-    <material name="silver"/>
-  </visual>
-  <!-- <collision>
-    <origin xyz="-0.015674 0.051597 -0.486315" rpy="0 0 0"/>
-    <geometry>
-      <mesh filename="file://$(find darnetnew_description)/meshes/MX-28AT_AR_6.stl" scale="0.001 0.001 0.001"/>
-    </geometry>
-  </collision> -->
-</link>
-<link name="14_FR07_S101_3">
-  <inertial>
-    <origin xyz="0.012032947663707046 0.01499993245518745 -0.003785284890375329" rpy="0 0 0"/>
-    <mass value="0.0014582156856158806"/>
-    <inertia ixx="0.0" iyy="0.0" izz="0.0" ixy="-0.0" iyz="0.0" ixz="0.0"/>
-  </inertial>
-  <visual>
-    <origin xyz="-0.007174 0.087097 -0.450515" rpy="0 0 0"/>
-    <geometry>
-      <mesh filename="file://$(find darnetnew_description)/meshes/14_FR07_S101_3.stl" scale="0.001 0.001 0.001"/>
-    </geometry>
-    <material name="silver"/>
-  </visual>
-  <!-- <collision>
-    <origin xyz="-0.007174 0.087097 -0.450515" rpy="0 0 0"/>
-    <geometry>
-      <mesh filename="file://$(find darnetnew_description)/meshes/14_FR07_S101_3.stl" scale="0.001 0.001 0.001"/>
-    </geometry>
-  </collision> -->
-</link>
-<link name="Hex_Spacer_MF_M3_L40mm_7">
-  <inertial>
-    <origin xyz="-0.011896 0.064319 -0.444515" rpy="0 0 0"/>
-    <mass value="0.01"/>
-    <inertia ixx="1e-6" iyy="1e-6" izz="1e-6" ixy="0" iyz="0" ixz="0"/>
-  </inertial>
-  <visual>
-    <origin xyz="-0.011896 0.064319 -0.444515" rpy="0 0 0"/>
-    <geometry>
-      <mesh filename="file://$(find darnetnew_description)/meshes/Hex_Spacer_MF_M3_L40mm_7.stl" scale="0.001 0.001 0.001"/>
-    </geometry>
-    <material name="silver"/>
-  </visual>
-  <!-- <collision>
-    <origin xyz="-0.011896 0.064319 -0.444515" rpy="0 0 0"/>
-    <geometry>
-      <mesh filename="file://$(find darnetnew_description)/meshes/Hex_Spacer_MF_M3_L40mm_7.stl" scale="0.001 0.001 0.001"/>
-    </geometry>
-  </collision> -->
-</link>
-<link name="Hex_Spacer_MF_M3_L40mm_6">
-  <inertial>
-    <origin xyz="-0.011896 0.079875 -0.444515" rpy="0 0 0"/>
-    <mass value="0.01"/>
-    <inertia ixx="1e-6" iyy="1e-6" izz="1e-6" ixy="0" iyz="0" ixz="0"/>
-  </inertial>
-  <visual>
-    <origin xyz="-0.011896 0.079875 -0.444515" rpy="0 0 0"/>
-    <geometry>
-      <mesh filename="file://$(find darnetnew_description)/meshes/Hex_Spacer_MF_M3_L40mm_6.stl" scale="0.001 0.001 0.001"/>
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