Commit message: Optimize mesh amam beberapa adjustment

File: src/darnet_controller_test/urdf/darnetnew.xacro (robot description, xacro)
@@ -8,5 +8,5 @@
     <inertial>
       <origin xyz="0.11490191942179352 -0.08811411521808868 0.4285754030138091" rpy="0 0 0"/>
-      <mass value="0.04783342981131993"/>
+      <mass value="1.34928"/>
       <inertia ixx="0.00012" iyy="0.000191" izz="0.00024" ixy="0.0" iyz="0.0" ixz="-0.0"/>
     </inertial>
@@ -168,5 +168,5 @@
     <inertial>
       <origin xyz="-4.036340476298861e-07 -0.0037563467783642973 -0.010402605928093445" rpy="0 0 0"/>
-      <mass value="0.008519664111309755"/>
+      <mass value="0.07430625"/>
       <inertia ixx="6e-06" iyy="2e-06" izz="6e-06" ixy="-0.0" iyz="0.0" ixz="0.0"/>
     </inertial>
@@ -192,5 +192,5 @@
     <inertial>
       <origin xyz="-4.0363404811560866e-07 -0.003756346778364089 -0.010402605928093445" rpy="0 0 0"/>
-      <mass value="0.008519664111309755"/>
+      <mass value="0.07430625"/>
       <inertia ixx="6e-06" iyy="2e-06" izz="6e-06" ixy="-0.0" iyz="0.0" ixz="0.0"/>
     </inertial>
@@ -314,8 +314,9 @@
     <inertial>
       <origin xyz="-2.2100633829229277e-05 -0.020219638153982887 -0.011283313957089425" rpy="0 0 0"/>
-      <mass value="0.0439903769719111"/>
+      <mass value="0.0576525"/>
       <inertia ixx="1.3e-05" iyy="1e-05" izz="8e-06" ixy="0.0" iyz="-0.0" ixz="-0.0"/>
     </inertial>
     <visual>
+      <!-- <origin xyz="-0.015674 0.0758 -0.51712" rpy="0 0 0"/> -->
       <origin xyz="-0.015674 0.051597 -0.486315" rpy="0 0 0"/>
       <geometry>
@@ -338,4 +339,5 @@
     </inertial>
     <visual>
+      <!-- <origin xyz="-0.007174 0.110940 -0.481320" rpy="0 0 0"/> -->
       <origin xyz="-0.007174 0.087097 -0.450515" rpy="0 0 0"/>
       <geometry>
@@ -358,5 +360,5 @@
       <material name="silver"/>
     </visual>
-</link>
+  </link>
   <link name="Hex_Spacer_MF_M3_L40mm_6">
     <inertial>
@@ -372,5 +374,5 @@
       <material name="silver"/>
     </visual>
-</link>
+  </link>
   <link name="Hex_Spacer_MF_M3_L40mm_8">
     <inertial>
@@ -386,5 +388,5 @@
       <material name="silver"/>
     </visual>
-</link>
+  </link>
   <link name="Hex_Spacer_MF_M3_L40mm_5">
     <inertial>
@@ -400,5 +402,5 @@
       <material name="silver"/>
     </visual>
-</link>
+  </link>
   <link name="14_FR07_S101_4">
     <inertial>
@@ -409,4 +411,5 @@
     <visual>
       <origin xyz="-0.011896 0.064319 -0.404515" rpy="0 0 0"/>
+      <!-- <origin xyz="-0.011896 0.064319 -0.404515" rpy="0 0 0"/> -->
       <geometry>
         <mesh filename="file://$(find darnetnew_description)/meshes/14_FR07_S101_4.stl" scale="0.001 0.001 0.001"/>
@@ -418,8 +421,9 @@
     <inertial>
       <origin xyz="0.014339927512303688 0.0012164395485890697 -0.01497736351351936" rpy="0 0 0"/>
-      <mass value="0.0439903769719111"/>
+      <mass value="0.0576525"/>
       <inertia ixx="1e-05" iyy="8e-06" izz="1.3e-05" ixy="0.0" iyz="0.0" ixz="0.0"/>
     </inertial>
     <visual>
+      <!-- <origin xyz="-0.004674 0.087440 -0.429320" rpy="0 0 0"/> -->
       <origin xyz="-0.004674 0.063597 -0.398515" rpy="0 0 0"/>
       <geometry>
@@ -442,4 +446,6 @@
     </inertial>
     <visual>
+      <!-- <origin xyz="0.004056 0.07494 -0.414320" rpy="0 0 0"/> -->
+      <!-- <origin xyz="0.004056 0.07494 -0.383515" rpy="0 0 0"/> -->
       <origin xyz="0.004056 0.051097 -0.383515" rpy="0 0 0"/>
       <geometry>
@@ -456,4 +462,5 @@
     </inertial>
     <visual>
+      <!-- <origin xyz="-0.018444 0.090940 -0.389820" rpy="0 0 0"/> -->
       <origin xyz="-0.018444 0.067097 -0.359015" rpy="0 0 0"/>
       <geometry>
@@ -470,4 +477,5 @@
     </inertial>
     <visual>
+      <!-- <origin xyz="-0.005944 0.090940 -0.370820" rpy="0 0 0"/> -->
       <origin xyz="-0.005944 0.067097 -0.340015" rpy="0 0 0"/>
       <geometry>
@@ -520,5 +528,5 @@
     <inertial>
       <origin xyz="-2.262154435872521e-05 -0.023069638153982427 -0.01128331395708665" rpy="0 0 0"/>
-      <mass value="0.0439903769719111"/>
+      <mass value="0.0576525"/>
       <inertia ixx="1.3e-05" iyy="1e-05" izz="8e-06" ixy="0.0" iyz="-0.0" ixz="-0.0"/>
     </inertial>
@@ -672,5 +680,5 @@
     <inertial>
       <origin xyz="0.015280265219602435 0.01821643954858139 -0.015022278423608926" rpy="0 0 0"/>
-      <mass value="0.0439903769719111"/>
+      <mass value="0.0576525"/>
       <inertia ixx="1e-05" iyy="8e-06" izz="1.3e-05" ixy="-0.0" iyz="-0.0" ixz="0.0"/>
     </inertial>
@@ -692,5 +700,5 @@
     <inertial>
       <origin xyz="-4.03759651407265e-07 -0.024847556106279797 -0.015203256663834375" rpy="0 0 0"/>
-      <mass value="0.07240225558380499"/>
+      <mass value="0.07430625"/>
       <inertia ixx="3e-05" iyy="2.5e-05" izz="1.7e-05" ixy="-0.0" iyz="-1e-06" ixz="-0.0"/>
     </inertial>
@@ -740,5 +748,5 @@
     <inertial>
       <origin xyz="-0.01745265453539349 0.017300192866770245 0.002796743336166141" rpy="0 0 0"/>
-      <mass value="0.07240225558380499"/>
+      <mass value="0.07430625"/>
       <inertia ixx="2.5e-05" iyy="3e-05" izz="1.7e-05" ixy="0.0" iyz="-0.0" ixz="1e-06"/>
     </inertial>
@@ -760,5 +768,5 @@
     <inertial>
       <origin xyz="0.02549983591096161 1.9299231801550576e-07 -0.04693927260375347" rpy="0 0 0"/>
-      <mass value="0.009633598501165654"/>
+      <mass value="0.07430625"/>
       <inertia ixx="7e-06" iyy="1e-05" izz="5e-06" ixy="-0.0" iyz="0.0" ixz="-0.0"/>
     </inertial>
@@ -794,5 +802,5 @@
     <inertial>
       <origin xyz="-4.037596519901321e-07 -0.02484755610627938 -0.015203256663834097" rpy="0 0 0"/>
-      <mass value="0.07240225558380499"/>
+      <mass value="0.07430625"/>
       <inertia ixx="3e-05" iyy="2.5e-05" izz="1.7e-05" ixy="-0.0" iyz="-1e-06" ixz="-0.0"/>
     </inertial>
@@ -842,5 +850,5 @@
     <inertial>
       <origin xyz="-0.016548152732702284 0.01730019311797787 0.0027967433361663074" rpy="0 0 0"/>
-      <mass value="0.07240225558380499"/>
+      <mass value="0.07430625"/>
       <inertia ixx="2.5e-05" iyy="3e-05" izz="1.7e-05" ixy="0.0" iyz="0.0" ixz="-1e-06"/>
     </inertial>
@@ -862,5 +870,5 @@
     <inertial>
       <origin xyz="-0.025500643178509308 1.929923183069393e-07 -0.04693927260375297" rpy="0 0 0"/>
-      <mass value="0.009633598501165654"/>
+      <mass value="0.07430625"/>
       <inertia ixx="7e-06" iyy="1e-05" izz="5e-06" ixy="-0.0" iyz="0.0" ixz="-0.0"/>
     </inertial>
@@ -1036,5 +1044,5 @@
     <inertial>
       <origin xyz="0.017452607722562546 0.011000192866771133 -0.030096589352505865" rpy="0 0 0"/>
-      <mass value="0.07240225558380499"/>
+      <mass value="0.07430625"/>
       <inertia ixx="2.5e-05" iyy="3e-05" izz="1.7e-05" ixy="-0.0" iyz="0.0" ixz="1e-06"/>
     </inertial>
@@ -1056,5 +1064,5 @@
     <inertial>
       <origin xyz="0.025500075455422044 0.010088786747853684 -0.048147731418395734" rpy="0 0 0"/>
-      <mass value="0.019905401683360396"/>
+      <mass value="0.297225"/>
       <inertia ixx="3.2e-05" iyy="3.8e-05" izz="1.4e-05" ixy="-0.0" iyz="-5e-06" ixz="-0.0"/>
     </inertial>
@@ -1076,5 +1084,5 @@
     <inertial>
       <origin xyz="-0.025499882723518774 0.010088786747854198 -0.048147779594986645" rpy="0 0 0"/>
-      <mass value="0.019905401683360396"/>
+      <mass value="0.297225"/>
       <inertia ixx="3.2e-05" iyy="3.8e-05" izz="1.4e-05" ixy="-0.0" iyz="-5e-06" ixz="-0.0"/>
     </inertial>
@@ -1096,5 +1104,5 @@
     <inertial>
       <origin xyz="0.024847585009340478 1.9311797885834814e-07 0.01520377916764483" rpy="0 0 0"/>
-      <mass value="0.07240225558380499"/>
+      <mass value="0.07430625"/>
       <inertia ixx="2.5e-05" iyy="3e-05" izz="1.7e-05" ixy="-0.0" iyz="-0.0" ixz="-1e-06"/>
     </inertial>
@@ -1116,5 +1124,5 @@
     <inertial>
       <origin xyz="-0.024847392277437513 1.9286677170604616e-07 0.015203730991054168" rpy="0 0 0"/>
-      <mass value="0.07240225558380499"/>
+      <mass value="0.07430625"/>
       <inertia ixx="2.5e-05" iyy="3e-05" izz="1.7e-05" ixy="-0.0" iyz="0.0" ixz="1e-06"/>
     </inertial>
@@ -1136,5 +1144,5 @@
     <inertial>
       <origin xyz="-0.017452414990658444 0.011000193117978355 -0.030096541175914426" rpy="0 0 0"/>
-      <mass value="0.07240225558380499"/>
+      <mass value="0.07430625"/>
       <inertia ixx="2.5e-05" iyy="3e-05" izz="1.7e-05" ixy="-0.0" iyz="-0.0" ixz="-1e-06"/>
     </inertial>
@@ -1252,5 +1260,5 @@
     <inertial>
       <origin xyz="3.56821216254688e-07 0.02909665322163736 -0.028141919744686078" rpy="0 0 0"/>
-      <mass value="0.008519664111309755"/>
+      <mass value="0.07430625"/>
       <inertia ixx="6.16e-06" iyy="2.13e-06" izz="5.95e-06" ixy="0.0" iyz="0.0" ixz="0.0"/>
     </inertial>
@@ -1272,5 +1280,5 @@
     <inertial>
       <origin xyz="-1.64089313414717e-07 0.02909665322163725 -0.028141871568095007" rpy="0 0 0"/>
-      <mass value="0.008519664111309755"/>
+      <mass value="0.07430625"/>
       <inertia ixx="6.16e-06" iyy="2.13e-06" izz="5.95e-06" ixy="0.0" iyz="0.0" ixz="0.0"/>
     </inertial>
@@ -1793,5 +1801,7 @@
   </joint>
   <joint name="Bahu Tangan Kiri" type="continuous">
-    <origin xyz="-0.0225 -0.0045 0.015" rpy="0 0 0"/>
+    <!-- <origin xyz="-0.0225 0.019343 -0.015805" rpy="0 0 0"/> -->
+    <!-- <origin xyz="-0.0225 -0.0045 0.015" rpy="0 0 0"/> -->
+    <origin xyz="-0.0225 0.0205 -0.016" rpy="0 0 0"/>
     <parent link="10_FR07_H102_3"/>
     <child link="MX-28AT_AR_6"/>
@@ -2295,9 +2305,11 @@
   <joint name="Kepala Putar">
     <command_interface name="position">
-      <param name="min">-3.14159</param>
-      <param name="max">3.14159</param>
+      <param name="min">-1.5708</param>
+      <param name="max">1.5708</param>
     </command_interface>
     <state_interface name="position">
       <param name="initial_value">0</param>
+      <param name="min">-1.5708</param>
+      <param name="max">1.5708</param>
     </state_interface>
   </joint>

File: src/darnetnew_description/urdf/darnetnew.xacro (robot description, xacro)
@@ -2619,3 +2619,216 @@
   <child link="pull_16"/>
 </joint>
+<!-- ROS2 Control -->
+<ros2_control name="GazeboSystem" type="system">
+  <hardware>
+    <plugin>gazebo_ros2_control/GazeboSystem</plugin>
+  </hardware>
+  <!-- Joint 1 -->
+  <joint name="Leher Putar">
+    <command_interface name="position">
+      <param name="min">-3.14159</param>
+      <param name="max">3.14159</param>
+    </command_interface>
+    <state_interface name="position">
+      <param name="initial_value">0</param>
+    </state_interface>
+  </joint>
+  <!-- Joint 2 -->
+  <joint name="Kepala Putar">
+    <command_interface name="position">
+      <param name="min">-1.5708</param>
+      <param name="max">1.5708</param>
+    </command_interface>
+    <state_interface name="position">
+      <param name="initial_value">0</param>
+      <param name="min">-1.5708</param>
+      <param name="max">1.5708</param>
+    </state_interface>
+  </joint>
+  <!-- Joint 3 -->
+  <joint name="Paha Atas Kanan">
+    <command_interface name="position">
+      <param name="min">-3.14159</param>
+      <param name="max">3.14159</param>
+    </command_interface>
+    <state_interface name="position">
+      <param name="initial_value">0</param>
+    </state_interface>
+  </joint>
+  <!-- Joint 4 -->
+  <joint name="Paha Atas Kiri">
+    <command_interface name="position">
+      <param name="min">-3.14159</param>
+      <param name="max">3.14159</param>
+    </command_interface>
+    <state_interface name="position">
+      <param name="initial_value">0</param>
+    </state_interface>
+  </joint>
+  <!-- Joint 5 -->
+  <joint name="Paha Kanan Putar">
+    <command_interface name="position">
+      <param name="min">-3.14159</param>
+      <param name="max">3.14159</param>
+    </command_interface>
+    <state_interface name="position">
+      <param name="initial_value">0</param>
+    </state_interface>
+  </joint>
+  <!-- Joint 6 -->
+  <joint name="Paha Kiri Putar">
+    <command_interface name="position">
+      <param name="min">-3.14159</param>
+      <param name="max">3.14159</param>
+    </command_interface>
+    <state_interface name="position">
+      <param name="initial_value">0</param>
+    </state_interface>
+  </joint>
+  <!-- Joint 7 -->
+  <joint name="Paha Bawah Kanan">
+    <command_interface name="position">
+      <param name="min">-3.14159</param>
+      <param name="max">3.14159</param>
+    </command_interface>
+    <state_interface name="position">
+      <param name="initial_value">0</param>
+    </state_interface>
+  </joint>
+  <!-- Joint 8 -->
+  <joint name="Paha Bawah Kiri">
+    <command_interface name="position">
+      <param name="min">-3.14159</param>
+      <param name="max">3.14159</param>
+    </command_interface>
+    <state_interface name="position">
+      <param name="initial_value">0</param>
+    </state_interface>
+  </joint>
+  <!-- Joint 9 -->
+  <joint name="Lutut Kanan">
+    <command_interface name="position">
+      <param name="min">-3.14159</param>
+      <param name="max">3.14159</param>
+    </command_interface>
+    <state_interface name="position">
+      <param name="initial_value">0</param>
+    </state_interface>
+  </joint>
+  <!-- Joint 10 -->
+  <joint name="Lutut Kiri">
+    <command_interface name="position">
+      <param name="min">-3.14159</param>
+      <param name="max">3.14159</param>
+    </command_interface>
+    <state_interface name="position">
+      <param name="initial_value">0</param>
+    </state_interface>
+  </joint>
+  <!-- Joint 11 -->
+  <joint name="Kaki Kanan Atas">
+    <command_interface name="position">
+      <param name="min">-3.14159</param>
+      <param name="max">3.14159</param>
+    </command_interface>
+    <state_interface name="position">
+      <param name="initial_value">0</param>
+    </state_interface>
+  </joint>
+  <!-- Joint 12 -->
+  <joint name="Kaki Kiri Atas">
+    <command_interface name="position">
+      <param name="min">-3.14159</param>
+      <param name="max">3.14159</param>
+    </command_interface>
+    <state_interface name="position">
+      <param name="initial_value">0</param>
+    </state_interface>
+  </joint>
+  <!-- Joint 13 -->
+  <joint name="Kaki Kanan Bawah">
+    <command_interface name="position">
+      <param name="min">-3.14159</param>
+      <param name="max">3.14159</param>
+    </command_interface>
+    <state_interface name="position">
+      <param name="initial_value">0</param>
+    </state_interface>
+  </joint>
+  <!-- Joint 14 -->
+  <joint name="Kaki Kiri Bawah">
+    <command_interface name="position">
+      <param name="min">-3.14159</param>
+      <param name="max">3.14159</param>
+    </command_interface>
+    <state_interface name="position">
+      <param name="initial_value">0</param>
+    </state_interface>
+  </joint>
+  <!-- Joint 15 -->
+  <joint name="Lengan Kiri">
+    <command_interface name="position">
+      <param name="min">-3.14159</param>
+      <param name="max">3.14159</param>
+    </command_interface>
+    <state_interface name="position">
+      <param name="initial_value">0</param>
+    </state_interface>
+  </joint>
+  <!-- Joint 16 -->
+  <joint name="Bahu Tangan Kiri">
+    <command_interface name="position">
+      <param name="min">-3.14159</param>
+      <param name="max">3.14159</param>
+    </command_interface>
+    <state_interface name="position">
+      <param name="initial_value">0</param>
+    </state_interface>
+  </joint>
+  <!-- Joint 17 -->
+  <joint name="Tangan Kiri">
+    <command_interface name="position">
+      <param name="min">-3.14159</param>
+      <param name="max">3.14159</param>
+    </command_interface>
+    <state_interface name="position">
+      <param name="initial_value">0</param>
+    </state_interface>
+  </joint>
+  <!-- Joint 18 -->
+  <joint name="Lengan Kanan">
+    <command_interface name="position">
+      <param name="min">-3.14159</param>
+      <param name="max">3.14159</param>
+    </command_interface>
+    <state_interface name="position">
+      <param name="initial_value">0</param>
+    </state_interface>
+  </joint>
+  <!-- Joint 19 -->
+  <joint name="Bahu Tangan Kanan">
+    <command_interface name="position">
+      <param name="min">-3.14159</param>
+      <param name="max">3.14159</param>
+    </command_interface>
+    <state_interface name="position">
+      <param name="initial_value">0</param>
+    </state_interface>
+  </joint>
+  <!-- Joint 20 -->
+  <joint name="Tangan Kanan">
+    <command_interface name="position">
+      <param name="min">-3.14159</param>
+      <param name="max">3.14159</param>
+    </command_interface>
+    <state_interface name="position">
+      <param name="initial_value">0</param>
+    </state_interface>
+  </joint>
+</ros2_control>
+<gazebo>
+  <plugin filename="libgazebo_ros2_control.so" name="gazebo_ros2_control">
+    <parameters>$(find darnetnew_description)/config/joint_controller.yaml</parameters>
+  </plugin>
+</gazebo>
 </robot>
