Commit message: added inverse kinematics in the darnet_description folder

File: src/darnet_description/urdf/darnet.xacro (robot description, xacro)
@@ -424,5 +424,43 @@
   </collision>
 </link>
-<joint name="Leher Putar" type="continuous">
+<link name="End_Effector_Tangan_Kanan_1">
+  <inertial>
+    <origin xyz="0 0 0" rpy="0 0 0"/>
+    <mass value="0.001"/> <inertia ixx="0.0001" iyy="0.0001" izz="0.0001" ixy="0" iyz="0" ixz="0"/>
+  </inertial>
+</link>
+<link name="End_Effector_Kaki_Kanan_1">
+  <inertial>
+    <origin xyz="0 0 0" rpy="0 0 0"/>
+    <mass value="0.001"/>
+    <inertia ixx="0.0001" iyy="0.0001" izz="0.0001" ixy="0" iyz="0" ixz="0"/>
+  </inertial>
+  <visual>
+    <origin xyz="0 0 0" rpy="0 0 0"/>
+    <geometry>
+       <box size="0.01 0.01 0.01"/>
+    </geometry>
+    <material name="blue">
+        <color rgba="0 0 1 0.5"/>
+    </material>
+  </visual>
+</link>
+<link name="End_Effector_Kaki_Kiri_1">
+  <inertial>
+    <origin xyz="0 0 0" rpy="0 0 0"/>
+    <mass value="0.001"/>
+    <inertia ixx="0.0001" iyy="0.0001" izz="0.0001" ixy="0" iyz="0" ixz="0"/>
+  </inertial>
+  <visual>
+    <origin xyz="0 0 0" rpy="0 0 0"/>
+    <geometry>
+       <box size="0.01 0.01 0.01"/>
+    </geometry>
+    <material name="blue">
+        <color rgba="0 0 1 0.5"/>
+    </material>
+  </visual>
+</link>
+<joint name="Leher Putar" type="revolute">
   <origin xyz="0.125659 -0.060429 0.520233" rpy="0 0 0"/>
   <parent link="base_link"/>
@@ -430,7 +468,7 @@
   <axis xyz="0.0 0.0 -1.0"/>
   <dynamics damping="0.5"/>
-  <limit effort="10" velocity="6"/>
-</joint>
-<joint name="Kepala Putar" type="continuous">
+  <limit lower="-3.14159" upper="3.14159"  effort="10" velocity="6"/>
+</joint>
+<joint name="Kepala Putar" type="revolute">
   <origin xyz="0.0225 0.0 0.028" rpy="0 0 0"/>
   <parent link="Konektor_Leher_1"/>
@@ -438,7 +476,7 @@
   <axis xyz="-1.0 -0.0 -0.0"/>
   <dynamics damping="0.5"/>
-  <limit effort="10" velocity="6"/>
-</joint>
-<joint name="Lengan Kiri" type="continuous">
+  <limit lower="-3.14159" upper="3.14159"  effort="10" velocity="6"/>
+</joint>
+<joint name="Lengan Kiri" type="revolute">
   <origin xyz="0.048157 -0.060473 0.495956" rpy="0 0 0"/>
   <parent link="base_link"/>
@@ -446,7 +484,7 @@
   <axis xyz="1.0 0.000471 0.0"/>
   <dynamics damping="1.5"/>
-  <limit effort="10" velocity="6"/>
-</joint>
-<joint name="Bahu Tangan Kiri" type="continuous">
+  <limit lower="-3.14159" upper="3.14159"  effort="10" velocity="6"/>
+</joint>
+<joint name="Bahu Tangan Kiri" type="revolute">
   <origin xyz="-0.02251 0.02249 -0.016" rpy="0 0 0"/>
   <parent link="Konektor_Bahu__3"/>
@@ -454,7 +492,7 @@
   <axis xyz="-0.000471 1.0 0.0"/>
   <dynamics damping="1.5"/>
-  <limit effort="10" velocity="6"/>
-</joint>
-<joint name="Tangan Kiri" type="continuous">
+  <limit lower="-3.14159" upper="3.14159"  effort="10" velocity="6"/>
+</joint>
+<joint name="Tangan Kiri" type="revolute">
   <origin xyz="-0.023341 -0.019361 -0.1028" rpy="0 0 0"/>
   <parent link="Lengan_Kiri_1"/>
@@ -462,7 +500,7 @@
   <axis xyz="1.0 0.000471 0.0"/>
   <dynamics damping="0.3"/>
-  <limit effort="10" velocity="6"/>
-</joint>
-<joint name="Lengan Kanan " type="continuous">
+  <limit lower="-3.14159" upper="3.14159"  effort="10" velocity="6"/>
+</joint>
+<joint name="Lengan Kanan" type="revolute">
   <origin xyz="0.202784 -0.0604 0.495956" rpy="0 0 0"/>
   <parent link="base_link"/>
@@ -470,7 +508,7 @@
   <axis xyz="-1.0 -0.000471 -0.0"/>
   <dynamics damping="1.5"/>
-  <limit effort="10" velocity="6"/>
-</joint>
-<joint name="Bahu Tangan Kanan" type="continuous">
+  <limit lower="-3.14159" upper="3.14159"  effort="10" velocity="6"/>
+</joint>
+<joint name="Bahu Tangan Kanan" type="revolute">
   <origin xyz="0.022489 0.022511 -0.016" rpy="0 0 0"/>
   <parent link="Konektor_Bahu__1"/>
@@ -478,7 +516,7 @@
   <axis xyz="0.000471 -1.0 -0.0"/>
   <dynamics damping="1.5"/>
-  <limit effort="10" velocity="6"/>
-</joint>
-<joint name="Tangan Kanan" type="continuous">
+  <limit lower="-3.14159" upper="3.14159"  effort="10" velocity="6"/>
+</joint>
+<joint name="Tangan Kanan" type="revolute">
   <origin xyz="0.023359 -0.019339 -0.1028" rpy="0 0 0"/>
   <parent link="Lengan_Kanan_1"/>
@@ -486,7 +524,7 @@
   <axis xyz="-1.0 -0.000471 -0.0"/>
   <dynamics damping="0.3"/>
-  <limit effort="10" velocity="6"/>
-</joint>
-<joint name="Paha Kiri Putar" type="continuous">
+  <limit lower="-3.14159" upper="3.14159" effort="10" velocity="6"/>
+</joint>
+<joint name="Paha Kiri Putar" type="revolute">
   <origin xyz="0.078463 -0.069966 0.351036" rpy="0 0 0"/>
   <parent link="base_link"/>
@@ -494,7 +532,7 @@
   <axis xyz="-0.0 -0.0 1.0"/>
   <dynamics damping="5.0"/>
-  <limit effort="40" velocity="6"/>
-</joint>
-<joint name="Paha Atas Kanan" type="continuous">
+  <limit lower="-3.14159" upper="3.14159"  effort="40" velocity="6"/>
+</joint>
+<joint name="Paha Atas Kanan" type="revolute">
   <origin xyz="0.172863 -0.069922 0.351036" rpy="0 0 0"/>
   <parent link="base_link"/>
@@ -502,7 +540,7 @@
   <axis xyz="-0.0 -0.0 1.0"/>
   <dynamics damping="5.0"/>
-  <limit effort="40" velocity="6"/>
-</joint>
-<joint name="Paha Kanan Putar" type="continuous">
+  <limit lower="-3.14159" upper="3.14159"  effort="40" velocity="6"/>
+</joint>
+<joint name="Paha Kanan Putar" type="revolute">
   <origin xyz="0.0 -0.032853 -0.036545" rpy="0 0 0"/>
   <parent link="Paha_Atas_3"/>
@@ -510,7 +548,7 @@
   <axis xyz="0.0 -1.0 -0.0"/>
   <dynamics damping="5.0"/>
-  <limit effort="40" velocity="6"/>
-</joint>
-<joint name="Paha Atas Kiri" type="continuous">
+  <limit lower="-3.14159" upper="3.14159"  effort="40" velocity="6"/>
+</joint>
+<joint name="Paha Atas Kiri" type="revolute">
   <origin xyz="0.0 -0.032853 -0.036545" rpy="0 0 0"/>
   <parent link="Paha_Atas_4"/>
@@ -518,7 +556,7 @@
   <axis xyz="0.0 -1.0 -0.0"/>
   <dynamics damping="5.0"/>
-  <limit effort="40" velocity="6"/>
-</joint>
-<joint name="Paha Bawah Kiri " type="continuous">
+  <limit lower="-3.14159" upper="3.14159"  effort="40" velocity="6"/>
+</joint>
+<joint name="Paha Bawah Kiri" type="revolute">
   <origin xyz="0.0253 0.0264 0.0" rpy="0 0 0"/>
   <parent link="Paha_Kiri_1"/>
@@ -526,7 +564,7 @@
   <axis xyz="-1.0 0.0 -0.0"/>
   <dynamics damping="3.0"/>
-  <limit effort="55" velocity="6"/>
-</joint>
-<joint name="Paha Bawah Kanan " type="continuous">
+  <limit lower="-3.14159" upper="3.14159"  effort="55" velocity="6"/>
+</joint>
+<joint name="Paha Bawah Kanan" type="revolute">
   <origin xyz="-0.0253 0.0264 0.0" rpy="0 0 0"/>
   <parent link="Paha_Kanan_1"/>
@@ -534,7 +572,7 @@
   <axis xyz="1.0 0.0 0.0"/>
   <dynamics damping="3.0"/>
-  <limit effort="55" velocity="6"/>
-</joint>
-<joint name="Lutut Kiri" type="continuous">
+  <limit lower="-3.14159" upper="3.14159"  effort="55" velocity="6"/>
+</joint>
+<joint name="Lutut Kiri" type="revolute">
   <origin xyz="-0.0002 0.0 -0.1228" rpy="0 0 0"/>
   <parent link="Lutut_Kiri__1"/>
@@ -542,7 +580,7 @@
   <axis xyz="-1.0 -0.0 -0.0"/>
   <dynamics damping="3.0"/>
-  <limit effort="55" velocity="6"/>
-</joint>
-<joint name="Lutut Kanan" type="continuous">
+  <limit lower="-3.14159" upper="3.14159"  effort="55" velocity="6"/>
+</joint>
+<joint name="Lutut Kanan" type="revolute">
   <origin xyz="0.000201 0.0 -0.123" rpy="0 0 0"/>
   <parent link="Lutut_Kanan_1"/>
@@ -550,7 +588,7 @@
   <axis xyz="1.0 0.0 0.0"/>
   <dynamics damping="3.0"/>
-  <limit effort="55" velocity="6"/>
-</joint>
-<joint name="Kaki Kiri Atas" type="continuous">
+  <limit lower="-3.14159" upper="3.14159"  effort="55" velocity="6"/>
+</joint>
+<joint name="Kaki Kiri Atas" type="revolute">
   <origin xyz="0.0 0.0 -0.121129" rpy="0 0 0"/>
   <parent link="Betis_2"/>
@@ -558,7 +596,7 @@
   <axis xyz="-1.0 -0.0 -0.0"/>
   <dynamics damping="1.0"/>
-  <limit effort="25" velocity="6"/>
-</joint>
-<joint name="Kaki Kiri Bawah" type="continuous">
+  <limit lower="-3.14159" upper="3.14159"  effort="25" velocity="6"/>
+</joint>
+<joint name="Kaki Kiri Bawah" type="revolute">
   <origin xyz="-0.0253 -0.0264 0.0" rpy="0 0 0"/>
   <parent link="Mata_Kaki_Kiri_1"/>
@@ -566,7 +604,7 @@
   <axis xyz="0.0 -1.0 0.0"/>
   <dynamics damping="1.0"/>
-  <limit effort="25" velocity="6"/>
-</joint>
-<joint name="Kaki Kanan Atas" type="continuous">
+  <limit lower="-3.14159" upper="3.14159"  effort="25" velocity="6"/>
+</joint>
+<joint name="Kaki Kanan Atas" type="revolute">
   <origin xyz="0.0 0.0 -0.121129" rpy="0 0 0"/>
   <parent link="Betis_1"/>
@@ -574,7 +612,7 @@
   <axis xyz="1.0 0.0 0.0"/>
   <dynamics damping="1.0"/>
-  <limit effort="25" velocity="6"/>
-</joint>
-<joint name="Kaki Kanan Bawah" type="continuous">
+  <limit lower="-3.14159" upper="3.14159"  effort="25" velocity="6"/>
+</joint>
+<joint name="Kaki Kanan Bawah" type="revolute">
   <origin xyz="0.0253 -0.0264 0.0" rpy="0 0 0"/>
   <parent link="Mata_Kaki_Kanan_1"/>
@@ -582,5 +620,20 @@
   <axis xyz="0.0 -1.0 0.0"/>
   <dynamics damping="1.0"/>
-  <limit effort="25" velocity="6"/>
+  <limit lower="-3.14159" upper="3.14159"  effort="25" velocity="6"/>
+</joint>
+<joint name="joint_end_effector_kanan" type="fixed">
+  <parent link="Tangan_Kanan_1"/>
+  <child link="End_Effector_Tangan_Kanan_1"/>
+  <origin xyz="-0.005 -0.015 -0.15" rpy="0 0 0"/>
+</joint>
+<joint name="joint_tapak_kaki_kanan" type="fixed">
+  <parent link="Kaki_Kanan_1"/>
+  <child link="End_Effector_Kaki_Kanan_1"/>
+  <origin xyz="0.013 0.0325 -0.069" rpy="0 0 0"/>
+</joint>
+<joint name="joint_tapak_kaki_kiri" type="fixed">
+  <parent link="Kaki_Kiri_1"/>
+  <child link="End_Effector_Kaki_Kiri_1"/>
+  <origin xyz="-0.013 0.0325 -0.069" rpy="0 0 0"/>
 </joint>
 <!-- ROS2 Control -->

Commit message: added smoother walk in Testing and Testing2

File: src/darnet_description/urdf/darnet.xacro (robot description, xacro)
@@ -378,7 +378,9 @@
   </visual>
   <collision>
-    <origin xyz="-0.078263 0.102819 -0.070562" rpy="0 0 0"/>
-    <geometry>
-      <mesh filename="file://$(find darnet_description)/meshes/Kaki_Kiri_1.stl" scale="0.001 0.001 0.001"/>
+    <!-- <origin xyz="-0.078263 0.102819 -0.070562" rpy="0 0 0"/> -->
+    <origin xyz="-0.014 0.032 -0.0393" rpy="0 0 0"/>
+    <geometry>
+      <!-- <mesh filename="file://$(find darnet_description)/meshes/Kaki_Kiri_1.stl" scale="0.001 0.001 0.001"/> -->
+      <box size="0.1 0.135 0.0025"/>
     </geometry>
   </collision>
@@ -418,7 +420,9 @@
   </visual>
   <collision>
-    <origin xyz="-0.173064 0.102775 -0.070362" rpy="0 0 0"/>
-    <geometry>
-      <mesh filename="file://$(find darnet_description)/meshes/Kaki_Kanan_1.stl" scale="0.001 0.001 0.001"/>
+    <!-- <origin xyz="-0.173064 0.102775 -0.070362" rpy="0 0 0"/> -->
+    <origin xyz="0.014 0.032 -0.0393" rpy="0 0 0"/>
+    <geometry>
+      <!-- <mesh filename="file://$(find darnet_description)/meshes/Kaki_Kanan_1.stl" scale="0.001 0.001 0.001"/> -->
+      <box size="0.1 0.135 0.0025"/>
     </geometry>
   </collision>
@@ -429,12 +433,5 @@
     <mass value="0.001"/> <inertia ixx="0.0001" iyy="0.0001" izz="0.0001" ixy="0" iyz="0" ixz="0"/>
   </inertial>
-</link>
-<link name="End_Effector_Kaki_Kanan_1">
-  <inertial>
-    <origin xyz="0 0 0" rpy="0 0 0"/>
-    <mass value="0.001"/>
-    <inertia ixx="0.0001" iyy="0.0001" izz="0.0001" ixy="0" iyz="0" ixz="0"/>
-  </inertial>
-  <visual>
+    <visual>
     <origin xyz="0 0 0" rpy="0 0 0"/>
     <geometry>
@@ -446,5 +443,37 @@
   </visual>
 </link>
+<link name="End_Effector_Kaki_Kanan_1">
+  <inertial>
+    <origin xyz="0 0 0" rpy="0 0 0"/>
+    <mass value="0.001"/>
+    <inertia ixx="0.0001" iyy="0.0001" izz="0.0001" ixy="0" iyz="0" ixz="0"/>
+  </inertial>
+  <visual>
+    <origin xyz="0 0 0" rpy="0 0 0"/>
+    <geometry>
+       <box size="0.01 0.01 0.01"/>
+    </geometry>
+    <material name="blue">
+        <color rgba="0 0 1 0.5"/>
+    </material>
+  </visual>
+</link>
 <link name="End_Effector_Kaki_Kiri_1">
+  <inertial>
+    <origin xyz="0 0 0" rpy="0 0 0"/>
+    <mass value="0.001"/>
+    <inertia ixx="0.0001" iyy="0.0001" izz="0.0001" ixy="0" iyz="0" ixz="0"/>
+  </inertial>
+  <visual>
+    <origin xyz="0 0 0" rpy="0 0 0"/>
+    <geometry>
+       <box size="0.01 0.01 0.01"/>
+    </geometry>
+    <material name="blue">
+        <color rgba="0 0 1 0.5"/>
+    </material>
+  </visual>
+</link>
+<link name="End_Effector_Tangan_Kiri_1">
   <inertial>
     <origin xyz="0 0 0" rpy="0 0 0"/>
@@ -636,4 +665,9 @@
   <child link="End_Effector_Kaki_Kiri_1"/>
   <origin xyz="-0.013 0.0325 -0.069" rpy="0 0 0"/>
+</joint>
+<joint name="joint_end_effector_kiri" type="fixed">
+  <parent link="Tangan_Kiri_1"/>
+  <child link="End_Effector_Tangan_Kiri_1"/>
+  <origin xyz="0.005 -0.015 -0.15" rpy="0 0 0"/>
 </joint>
 <!-- ROS2 Control -->

Commit message: addded Jalan_Launcher and Coms for openRB

File: src/darnet_description/urdf/darnet.xacro (robot description, xacro)
@@ -491,4 +491,27 @@
   </visual>
 </link>
+<joint name="imu_joint" type="fixed">
+    <parent link="base_link"/>
+    <child link="imu_link"/>
+     <origin xyz="0.125659 -0.060429 0.4320233" rpy="0 0 0"/>
+  </joint>
+  <link name="imu_link">
+    <visual>
+      <geometry>
+        <box size="0.01 0.01 0.01"/> </geometry>
+      <material name="black">
+        <color rgba="0 0 0 1"/>
+      </material>
+    </visual>
+    <!-- <collision>
+      <geometry>
+        <box size="0.01 0.01 0.01"/>
+      </geometry>
+    </collision> -->
+    <inertial>
+      <mass value="0.01"/>
+      <inertia ixx="0.0001" ixy="0" ixz="0" iyy="0.0001" iyz="0" izz="0.0001"/>
+    </inertial>
+  </link>
 <joint name="Leher Putar" type="revolute">
   <origin xyz="0.125659 -0.060429 0.520233" rpy="0 0 0"/>
@@ -885,3 +908,18 @@
   <self_collide>1</self_collide>
 </gazebo>
+<gazebo reference="imu_link">
+    <sensor name="imu_sensor" type="imu">
+      <always_on>true</always_on>
+      <update_rate>100</update_rate> <visualize>true</visualize>
+      <plugin name="imu_plugin" filename="libgazebo_ros_imu_sensor.so">
+        <ros>
+          <namespace>/</namespace>
+          <remapping>~/out:=imu/data</remapping>
+        </ros>
+        <frame_name>imu_link</frame_name>
+        <initial_orientation_as_reference>false</initial_orientation_as_reference>
+      </plugin>
+      <pose>0 0 0 0 0 0</pose>
+    </sensor>
+  </gazebo>
 </robot>

Commit message: added imu sensor and camera to the simulation

File: src/darnet_description/urdf/darnet.xacro (robot description, xacro)
@@ -491,4 +491,5 @@
   </visual>
 </link>
+<!-- LINK SENSOR IMU -->
 <joint name="imu_joint" type="fixed">
     <parent link="base_link"/>
@@ -514,4 +515,35 @@
     </inertial>
   </link>
+<!-- LINK KAMERA -->
+<joint name="camera_joint" type="fixed">
+    <parent link="base_link"/>
+    <child link="camera_link"/>
+    <origin xyz="0.125659 -0.060429 0.6020233" rpy="0 0 1.5707"/>
+  </joint>
+  <link name="camera_link">
+    <visual>
+      <geometry>
+        <box size="0.02 0.05 0.02"/>
+      </geometry>
+      <material name="silver">
+        <color rgba="0.8 0.8 0.8 1"/>
+      </material>
+    </visual>
+    <collision>
+      <geometry>
+        <box size="0.02 0.05 0.02"/>
+      </geometry>
+    </collision>
+    <inertial>
+      <mass value="0.01"/>
+      <inertia ixx="0.0001" ixy="0" ixz="0" iyy="0.0001" iyz="0" izz="0.0001"/>
+    </inertial>
+  </link>
+  <joint name="camera_optical_joint" type="fixed">
+    <parent link="camera_link"/>
+    <child link="camera_link_optical"/>
+    <origin xyz="0 0 0" rpy="-1.5707 0 -1.5707"/>
+  </joint>
+  <link name="camera_link_optical"></link>
 <joint name="Leher Putar" type="revolute">
   <origin xyz="0.125659 -0.060429 0.520233" rpy="0 0 0"/>
@@ -901,4 +933,16 @@
     </state_interface>
   </joint>
+  <sensor name="imu_sensor">
+    <state_interface name="orientation.x"/>
+    <state_interface name="orientation.y"/>
+    <state_interface name="orientation.z"/>
+    <state_interface name="orientation.w"/>
+    <state_interface name="angular_velocity.x"/>
+    <state_interface name="angular_velocity.y"/>
+    <state_interface name="angular_velocity.z"/>
+    <state_interface name="linear_acceleration.x"/>
+    <state_interface name="linear_acceleration.y"/>
+    <state_interface name="linear_acceleration.z"/>
+  </sensor>
 </ros2_control>
 <gazebo>
@@ -911,6 +955,7 @@
     <sensor name="imu_sensor" type="imu">
       <always_on>true</always_on>
-      <update_rate>100</update_rate> <visualize>true</visualize>
-      <plugin name="imu_plugin" filename="libgazebo_ros_imu_sensor.so">
+      <update_rate>100</update_rate>
+      <visualize>true</visualize>
+      <plugin filename="libignition-gazebo-imu-system.so" name="ignition::gazebo::systems::Imu">
         <ros>
           <namespace>/</namespace>
@@ -922,4 +967,28 @@
       <pose>0 0 0 0 0 0</pose>
     </sensor>
+</gazebo>
+<gazebo reference="camera_link">
+    <sensor name="camera" type="camera">
+      <update_rate>30.0</update_rate>
+      <always_on>true</always_on>
+      <visualize>true</visualize>
+      <plugin filename="libignition-gazebo-sensors-system.so"
+            name="ignition::gazebo::systems::Sensors">
+        <render_engine>ogre2</render_engine>
+    </plugin>
+      <topic>camera/image_raw</topic>
+      <camera name="head">
+        <horizontal_fov>1.3962634</horizontal_fov>
+        <image>
+          <width>640</width>
+          <height>480</height>
+          <format>R8G8B8</format>
+        </image>
+        <clip>
+          <near>0.02</near>
+          <far>300</far>
+        </clip>
+      </camera>
+      </sensor>
   </gazebo>
 </robot>

Commit message: added new walking script

File: src/darnet_description/urdf/darnet.xacro (robot description, xacro)
@@ -24,4 +24,13 @@
   </collision>
 </link>
+<link name="base_center">
+    <visual>
+      <geometry>
+         <box size="0.01 0.01 0.01"/>
+      </geometry>
+      <material name="red"/>
+        <color rgba="1 0 0 0.5"/>
+    </visual>
+  </link>
 <link name="Konektor_Leher_1">
   <inertial>
@@ -517,7 +526,7 @@
 <!-- LINK KAMERA -->
 <joint name="camera_joint" type="fixed">
-    <parent link="base_link"/>
+    <parent link="Kepala_4"/>
     <child link="camera_link"/>
-    <origin xyz="0.125659 -0.060429 0.6020233" rpy="0 0 1.5707"/>
+    <origin xyz="-0.0225 0 0.05379" rpy="0 0 1.5707"/>
   </joint>
   <link name="camera_link">
@@ -546,4 +555,9 @@
   </joint>
   <link name="camera_link_optical"></link>
+<joint name="center_to_base" type="fixed">
+    <parent link="base_center"/>
+    <child link="base_link"/>
+    <origin xyz="-0.125659 0.060429 -0.03189" rpy="0 0 0"/>
+  </joint>
 <joint name="Leher Putar" type="revolute">
   <origin xyz="0.125659 -0.060429 0.520233" rpy="0 0 0"/>
@@ -714,10 +728,10 @@
   <parent link="Kaki_Kanan_1"/>
   <child link="End_Effector_Kaki_Kanan_1"/>
-  <origin xyz="0.013 0.0325 -0.069" rpy="0 0 0"/>
+  <origin xyz="0.013 0.0325 -0.04" rpy="0 0 0"/>
 </joint>
 <joint name="joint_tapak_kaki_kiri" type="fixed">
   <parent link="Kaki_Kiri_1"/>
   <child link="End_Effector_Kaki_Kiri_1"/>
-  <origin xyz="-0.013 0.0325 -0.069" rpy="0 0 0"/>
+  <origin xyz="-0.013 0.0325 -0.04" rpy="0 0 0"/>
 </joint>
 <joint name="joint_end_effector_kiri" type="fixed">
